Commit message: terabot_description: Changin ros_control xacro name

File: terabot_description/urdf/terabot.gazebo.xacro (robot description, xacro)
@@ -51,5 +51,5 @@
 	  </gazebo>
   </xacro:macro>
-  <xacro:macro name="ros_control" params="namespace">
+  <xacro:macro name="ros_control_terabot" params="namespace">
 		<gazebo>
 			<plugin name="ros_control" filename="libgazebo_ros_control.so">

File: terabot_description/urdf/terabot_standalone.urdf.xacro (robot description, xacro)
@@ -35,4 +35,4 @@
 	</link>
   <xacro:terabot name="terabot" parent="base_link" />
-  <xacro:ros_control namespace="/terabot"/>
+  <xacro:ros_control_terabot namespace="/terabot"/>
 </robot>
