Commit message: terabot_description: Corrected error in standalone urdf

File: terabot_description/urdf/terabot.urdf.xacro (robot description, xacro)
@@ -1,29 +1,28 @@
 <?xml version="1.0"?>
 <robot name="terabot" xmlns:xacro="http://www.ros.org/wiki/xacro">
-   <!-- TERABOT_ARM -->
-  <!-- Import all Gazebo-customization elements, including Gazebo colors -->
-  <xacro:include filename="$(find terabot_description)/urdf/terabot.gazebo.xacro" />
-  <!--xacro:include filename="$(find terabot_description)/urdf/tcp.urdf.xacro" /-->
-  <!-- Constants for robot dimensions -->
-  <xacro:property name="PI" value="3.1415926535897931"/>
-  <xacro:property name="j1_mechanical_reduction" value="250.0"/>
-  <xacro:property name="j1_motor_torque_constant" value="5.0"/>
-  <xacro:property name="j2_mechanical_reduction" value="250.0"/>
-  <xacro:property name="j2_motor_torque_constant" value="5.0"/>
-  <xacro:property name="j5_mechanical_reduction" value="250.0"/>
-  <xacro:property name="j5_motor_torque_constant" value="5.0"/>
-  <xacro:property name="j8_mechanical_reduction" value="1"/>
-  <xacro:property name="j8_motor_torque_constant" value="1"/>
-  <xacro:property name="j9_mechanical_reduction" value="250.0"/>
-  <xacro:property name="j9_motor_torque_constant" value="5.0"/>
-  <xacro:property name="finger_mechanical_reduction" value="1.0"/>
-  <xacro:property name="finger_motor_torque_constant" value="1.0"/>
-  <xacro:property name="joint_effort_limit" value="100.0"/>
-  <xacro:property name="joint_velocity_limit" value="3.0"/>
-  <xacro:property name="joint_damping" value="0.5"/>
-  <xacro:property name="joint_friction" value="0.5"/>
-  <xacro:macro name="terabot" params="parent name">
-	  <link
-		name="${name}_0_link">
+<!-- TERABOT_ARM -->
+<!-- Import all Gazebo-customization elements, including Gazebo colors -->
+<xacro:include filename="$(find terabot_description)/urdf/terabot.gazebo.xacro" />
+<!--xacro:include filename="$(find terabot_description)/urdf/tcp.urdf.xacro" /-->
+<!-- Constants for robot dimensions -->
+<xacro:property name="PI" value="3.1415926535897931"/>
+<xacro:property name="j1_mechanical_reduction" value="250.0"/>
+<xacro:property name="j1_motor_torque_constant" value="5.0"/>
+<xacro:property name="j2_mechanical_reduction" value="250.0"/>
+<xacro:property name="j2_motor_torque_constant" value="5.0"/>
+<xacro:property name="j5_mechanical_reduction" value="250.0"/>
+<xacro:property name="j5_motor_torque_constant" value="5.0"/>
+<xacro:property name="j8_mechanical_reduction" value="1"/>
+<xacro:property name="j8_motor_torque_constant" value="1"/>
+<xacro:property name="j9_mechanical_reduction" value="250.0"/>
+<xacro:property name="j9_motor_torque_constant" value="5.0"/>
+<xacro:property name="finger_mechanical_reduction" value="1.0"/>
+<xacro:property name="finger_motor_torque_constant" value="1.0"/>
+<xacro:property name="joint_effort_limit" value="100.0"/>
+<xacro:property name="joint_velocity_limit" value="3.0"/>
+<xacro:property name="joint_damping" value="0.5"/>
+<xacro:property name="joint_friction" value="0.5"/>
+<xacro:macro name="terabot" params="parent name">
+	  <link	name="${name}_0_link">
 		<inertial>
 		  <origin
@@ -64,7 +63,5 @@
 		</collision>
 	  </link>
-	  <joint
-		name="${name}_0_joint"
-		type="fixed">
+	  <joint name="${name}_0_joint"	type="fixed">
 		<origin
 		  xyz="0.0 0.0 0.0"
@@ -77,6 +74,5 @@
 		  xyz="0 0 0" />
 	  </joint>
-	  <link
-		name="${name}_1_link">
+	  <link name="${name}_1_link">
 		<inertial>
 		  <origin
@@ -118,7 +114,5 @@
 		</collision>
 	  </link>
-	  <joint
-		name="${name}_1_joint"
-		type="revolute">
+	  <joint name="${name}_1_joint" type="revolute">
 		<origin
 		  xyz="0 0 0.19178"
@@ -144,6 +138,5 @@
 		 </actuator>
 	  </transmission>
-	  <link
-		name="${name}_2_link">
+	  <link	name="${name}_2_link">
 		<inertial>
 		  <origin
@@ -185,7 +178,5 @@
 		</collision>
 	  </link>
-	  <joint
-		name="${name}_2_joint"
-		type="revolute">
+	  <joint name="${name}_2_joint"	type="revolute">
 		<origin
 		  xyz="0 0.00939800000000001 0"
@@ -197,5 +188,4 @@
 		<axis
 		  xyz="0 -1 0" />
-		<!-- limit effort="100" velocity="100" upper="0" lower="-1.6557984366"/ -->
 		<limit effort="${joint_effort_limit}" velocity="${joint_velocity_limit}" upper="0" lower="-2.094395102"/>
 		<dynamics damping="${joint_damping}" friction="${joint_friction}"/>
@@ -210,6 +200,5 @@
 		 </actuator>
 	  </transmission>
-	  <link
-		name="${name}_3_link">
+	  <link name="${name}_3_link">
 		<inertial>
 		  <origin
@@ -251,7 +240,5 @@
 		</collision>
 	  </link>
-	  <joint
-		name="${name}_3_joint"
-		type="fixed">
+	  <joint name="${name}_3_joint"	type="fixed">
 		<origin
 		  xyz="0.0526796 0 0.0351028"
@@ -264,6 +251,5 @@
 		  xyz="0 0 0" />
 	  </joint>
-	  <link
-		name="${name}_4_link">
+	  <link	name="${name}_4_link">
 		<inertial>
 		  <origin
@@ -305,7 +291,5 @@
 		</collision>
 	  </link>
-	  <joint
-		name="${name}_4_joint"
-		type="fixed">
+	  <joint name="${name}_4_joint" type="fixed">
 		<origin
 		  xyz="0.36642 0 -0.035103"
@@ -318,6 +302,5 @@
 		  xyz="0 0 0" />
 	  </joint>
-	  <link
-		name="${name}_5_link">
+	  <link	name="${name}_5_link">
 		<inertial>
 		  <origin
@@ -359,7 +342,5 @@
 		</collision>
 	  </link>
-	  <joint
-		name="${name}_5_joint"
-		type="revolute">
+	  <joint name="${name}_5_joint"	type="revolute">
 		<origin
 		  xyz="0 0.0582295 0"
@@ -371,5 +352,4 @@
 		<axis
 		  xyz="0 -1 0" />
-		<!-- limit effort="100" velocity="100" upper="2.96705" lower="-2.82743"/ -->
 		<limit effort="${joint_effort_limit}" velocity="${joint_velocity_limit}" upper="2.79208312055332" lower="-2.7928224140"/>
 		<dynamics damping="${joint_damping}" friction="${joint_friction}"/>
@@ -384,6 +364,5 @@
 		 </actuator>
 	  </transmission>
-	  <link
-		name="${name}_6_link">
+	  <link	name="${name}_6_link">
 		<inertial>
 		  <origin
@@ -425,7 +404,5 @@
 		</collision>
 	  </link>
-	  <joint
-		name="${name}_6_joint"
-		type="fixed">
+	  <joint name="${name}_6_joint"	type="fixed">
 		<origin
 		  xyz="0.04445 0 0.035103"
@@ -438,6 +415,5 @@
 		  xyz="0 0 0" />
 	  </joint>
-	  <link
-		name="${name}_7_link">
+	  <link	name="${name}_7_link">
 		<inertial>
 		  <origin
@@ -479,7 +455,5 @@
 		</collision>
 	  </link>
-	  <joint
-		name="${name}_7_joint"
-		type="fixed">
+	  <joint name="${name}_7_joint"	type="fixed">
 		<origin
 		  xyz="0.32009 0 -0.028753"
@@ -533,7 +507,5 @@
 		</collision>
 	  </link>
-	  <joint
-		name="${name}_8_joint"
-		type="revolute">
+	  <joint name="${name}_8_joint"	type="revolute">
 		<origin
 		  xyz="0 0.04699 0"
@@ -557,6 +529,5 @@
 		 </actuator>
 	  </transmission>
-	  <link
-		name="${name}_9_link">
+	  <link name="${name}_9_link">
 		<inertial>
 		  <origin
@@ -598,7 +569,5 @@
 		</collision>
 	  </link>
-	  <joint
-		name="${name}_9_joint"
-		type="revolute">
+	  <joint name="${name}_9_joint" type="revolute">
 		<origin
 		  xyz="0.0769366 0 0.0328168"
@@ -622,6 +591,5 @@
 		 </actuator>
 	  </transmission>
-	  <link
-		name="${name}_91_link">
+	  <link name="${name}_91_link">
 		<inertial>
 		  <origin
@@ -662,6 +630,5 @@
 		</collision>
 	  </link>
-	  <joint
-		name="${name}_91_joint"
+	  <joint name="${name}_91_joint"
 		type="revolute">
 		<origin
@@ -686,6 +653,5 @@
 		 </actuator>
 	  </transmission>
-	  <link
-		name="${name}_92_link">
+	  <link	name="${name}_92_link">
 		<inertial>
 		  <origin
@@ -726,7 +692,5 @@
 		</collision>
 	  </link>
-	  <joint
-		name="${name}_92_joint"
-		type="revolute">
+	  <joint name="${name}_92_joint" type="revolute">
 		<origin
 		  xyz="0.097993 -0.028575 0"
@@ -751,6 +715,6 @@
 	  </transmission>
 	<!-- extensions -->
-	<xacro:terabot_gazebo name="${name}" />
+	<!--xacro:terabot_gazebo name="${name}" /-->
 	<!-- TCP management -->
-  </xacro:macro>
+</xacro:macro>
 </robot>

File: terabot_description/urdf/terabot_standalone.urdf.xacro (robot description, xacro)
@@ -3,12 +3,13 @@
   <!-- Import all Gazebo-customization elements, including Gazebo colors -->
   <xacro:include filename="$(find terabot_description)/urdf/terabot.urdf.xacro" />
-  <xacro:include filename="$(find terabot_description)/urdf/terabot.gazebo.xacro" />
-  <!-- Used for fixing robot to Gazebo 'base_link' -->
+  <!--xacro:include filename="$(find terabot_description)/urdf/terabot.gazebo.xacro" /-->
   <link name="world"/>
-  <joint name="fwf" type="fixed">
-    <parent link="world"/>
-    <child link="base_footprint"/>
+  <joint name="fixed" type="fixed">
+	<parent link="world"/>
+	<child link="base_footprint"/>
   </joint>
   <!-- BASE FOOTPRINT -->
+  <!-- base_footprint is a fictitious link(frame) that is on the ground right below base_link origin,
+             navigation stack depends on this frame -->
   <link name="base_footprint">
       <visual>
@@ -26,10 +27,12 @@
   </link>
   <joint name="base_footprint_joint" type="fixed">
-     <!-- origin xyz="0 0 0.050" rpy="0 0 0" / -->
-     <origin xyz="0 0 0.50" rpy="0 0 0" />
+     <origin xyz="0 0 0" rpy="0 0 0" />
      <parent link="base_footprint"/>
-     <child link="terabot_0_link" />
+     <child link="base_link" />
   </joint>
-  <xacro:terabot name="terabot" parent="base_footprint" />
+	<!-- BASE_LINK (RED) -->
+	<link name="base_link">
+	</link>
+  <xacro:terabot name="terabot" parent="base_link" />
   <xacro:ros_control namespace="/terabot"/>
 </robot>

Commit message: terabot_description: Modifying limits

File: terabot_description/urdf/terabot.urdf.xacro (robot description, xacro)
@@ -20,5 +20,5 @@
 <xacro:property name="finger_motor_torque_constant" value="1.0"/>
 <xacro:property name="joint_effort_limit" value="100.0"/>
-<xacro:property name="joint_velocity_limit" value="3.0"/>
+<xacro:property name="joint_velocity_limit" value="0.61"/>
 <xacro:property name="joint_damping" value="0.5"/>
 <xacro:property name="joint_friction" value="0.5"/>

Commit message: terabot_description: Adding block origin to urdf.xacro

File: terabot_description/urdf/terabot.urdf.xacro (robot description, xacro)
@@ -23,5 +23,5 @@
 <xacro:property name="joint_damping" value="0.5"/>
 <xacro:property name="joint_friction" value="0.5"/>
-<xacro:macro name="terabot" params="parent name">
+<xacro:macro name="terabot" params="parent name *origin">
 	  <link	name="${name}_0_link">
 		<inertial>
@@ -64,7 +64,5 @@
 	  </link>
 	  <joint name="${name}_0_joint"	type="fixed">
-		<origin
-		  xyz="0.0 0.0 0.0"
-		  rpy="0.0 0.0 0.0" />
+		<insert_block name="origin" />
 		<parent
 		  link="${parent}" />

File: terabot_description/urdf/terabot_standalone.urdf.xacro (robot description, xacro)
@@ -34,5 +34,7 @@
 	<link name="base_link">
 	</link>
-  <xacro:terabot name="terabot" parent="base_link" />
+  <xacro:terabot name="terabot" parent="base_link">
+	  <origin xyz="0 0 0" rpy="0 0 0"/>
+  </xacro:terabot>
   <xacro:ros_control_terabot namespace="/terabot"/>
 </robot>
